File: DisplayController.sch (KiCad schematic (older format))
At the start: 0 parts

Commit message: modified:   DisplayController.sch 	modified:   KeypadController.sch 	new file:   QC2004A.kicad_mod 	modified:   RasPiInterface.lib 	modified:   RasPiInterface.sch 	new file:   Raspberry-I2C-LCD-and-Keypad-B_Cu.gbr 	new file:   Raspberry-I2C-LCD-and-Keypad-B_Mask.gbr 	new file:   Raspberry-I2C-LCD-and-Keypad-B_Paste.gbr 	new file:   Raspberry-I2C-LCD-and-Keypad-Edge_Cuts.gbr 	new file:   Raspberry-I2C-LCD-and-Keypad-F_Cu.gbr 	new file:   Raspberry-I2C-LCD-and-Keypad-F_Mask.gbr 	new file:   Raspberry-I2C-LCD-and-Keypad-F_Paste.gbr 	new file:   Raspberry-I2C-LCD-and-Keypad-F_SilkS.gbr 	new file:   Raspberry-I2C-LCD-and-Keypad-NPTH.drl 	new file:   Raspberry-I2C-LCD-and-Keypad-PTH.drl 	modified:   Raspberry-I2C-LCD-and-Keypad-cache.lib 	modified:   Raspberry-I2C-LCD-and-Keypad.kicad_pcb 	new file:   Raspberry-I2C-LCD-and-Keypad.kicad_pcb-bak 	modified:   Raspberry-I2C-LCD-and-Keypad.pro 	modified:   Raspberry-I2C-LCD-and-Keypad.sch 	modified:   fp-info-cache
Parts:
- added C1: 100n, Capacitor_THT:C_Disc_D5.0mm_W2.5mm_P2.50mm, symbol Device:C
- added C2: 10µ, Capacitor_THT:CP_Radial_Tantal_D4.5mm_P2.50mm, symbol Device:CP1
- added D1: green, LED_THT:LED_D3.0mm_Horizontal_O3.81mm_Z2.0mm, symbol Device:LED
- added JP1, JP2, JP3: Jumper_NC_Dual, Jumper:SolderJumper-3_P1.3mm_Open_RoundedPad1.0x1.5mm_NumberLabels, symbol Device:Jumper_NC_Dual
- added Q20: BC557, Package_TO_SOT_THT:TO-92_Horizontal1, symbol Device:Q_PNP_CBE
- added R1: 4k7, Resistor_THT:R_Axial_DIN0207_L6.3mm_D2.5mm_P7.62mm_Horizontal, symbol Device:R_US
- added R2: 1k, Resistor_THT:R_Axial_DIN0207_L6.3mm_D2.5mm_P7.62mm_Horizontal, symbol Device:R_US
- added R3: 180, Resistor_THT:R_Axial_DIN0207_L6.3mm_D2.5mm_P7.62mm_Horizontal, symbol Device:R_US
- added RV1: 10k, Potentiometer_THT:Potentiometer_Vishay_43_Horizontal, symbol Device:R_POT_TRIM_US
- added U20: PCF8574A, Package_DIP:DIP-16_W7.62mm, symbol Interface_Expansion:PCF8574A
- added U21: LCD_HD44780, Raspberry-I2C-LCD-and-Keypad:QC2004A, symbol RasPiInterface:LCD_HD44780
Connections:
- new net: U20.4 (P0), U21.11 (DB4/0)
- new net: U20.5 (P1), U21.12 (DB5/1)
- new net: U20.6 (P2), U21.13 (DB6/2)
- new net: U20.7 (P3), U21.14 (DB7/3)
- new net: R3.1, U21.15 (BL+)
- new net: RV1.2, U21.3 (VC)
- new net: U20.9 (P4), U21.4 (RS)
- new net: U20.10 (P5), U21.5 (R/~W)
- new net: U20.11 (P6), U21.6 (E)
- new net: JP1.2, U20.1 (A0)
- new net: R2.1, U20.12 (P7)
- new net: JP2.2, U20.2 (A1)
- new net: JP3.2, U20.3 (A2)
- new net: Q20.1 (C), R3.2
- new net: D1.2 (A), Q20.2 (B), R1.1
- new net: D1.1 (K), R2.2
- new net 3.3V: C1.2, JP1.3, JP2.3, JP3.3, U20.16 (VDD)
- new net 5V: C2.1, Q20.3 (E), R1.2, RV1.3, U21.2 (Vcc)
- new net GND: C1.1, C2.2, JP1.1, JP2.1, JP3.1, RV1.1, U20.8 (VSS), U21.1 (GND), U21.16 (BL-)
- new net SCL: U20.14 (SCL)
- new net SDA: U20.15 (SDA)
