File: KeypadController.sch (KiCad schematic (older format))
At the start: 6 parts, among them J10 Conn_01x08, J11 Conn_01x08, J12 Conn_01x08, U10 TCA8418

Commit message: modified:   DisplayController.sch 	modified:   KeypadController.sch 	new file:   QC2004A.kicad_mod 	modified:   RasPiInterface.lib 	modified:   RasPiInterface.sch 	new file:   Raspberry-I2C-LCD-and-Keypad-B_Cu.gbr 	new file:   Raspberry-I2C-LCD-and-Keypad-B_Mask.gbr 	new file:   Raspberry-I2C-LCD-and-Keypad-B_Paste.gbr 	new file:   Raspberry-I2C-LCD-and-Keypad-Edge_Cuts.gbr 	new file:   Raspberry-I2C-LCD-and-Keypad-F_Cu.gbr 	new file:   Raspberry-I2C-LCD-and-Keypad-F_Mask.gbr 	new file:   Raspberry-I2C-LCD-and-Keypad-F_Paste.gbr 	new file:   Raspberry-I2C-LCD-and-Keypad-F_SilkS.gbr 	new file:   Raspberry-I2C-LCD-and-Keypad-NPTH.drl 	new file:   Raspberry-I2C-LCD-and-Keypad-PTH.drl 	modified:   Raspberry-I2C-LCD-and-Keypad-cache.lib 	modified:   Raspberry-I2C-LCD-and-Keypad.kicad_pcb 	new file:   Raspberry-I2C-LCD-and-Keypad.kicad_pcb-bak 	modified:   Raspberry-I2C-LCD-and-Keypad.pro 	modified:   Raspberry-I2C-LCD-and-Keypad.sch 	modified:   fp-info-cache
Parts:
- removed RN1: R_Network06_US, Resistor_THT:R_Array_SIP7, symbol Device:R_Network06_US
- added RN1: 10k, Resistor_THT:R_Array_SIP9, symbol Device:R_Network08_US
- C5: renamed from C10; footprint Capacitor_THT:C_Disc_D5.0mm_W2.5mm_P2.50mm -> Capacitor_THT:C_Disc_D5.0mm_W2.5mm_P5.00mm
- J2: renamed from J10; footprint Connector_PinHeader_1.27mm:PinHeader_1x06_P1.27mm_Vertical -> Connector_PinHeader_1.27mm:PinHeader_1x08_P1.27mm_Horizontal
- J3: renamed from J12; footprint Connector_PinHeader_1.27mm:PinHeader_1x06_P1.27mm_Vertical -> Connector_PinHeader_1.27mm:PinHeader_1x08_P1.27mm_Horizontal
- J4: renamed from J11; footprint Connector_PinHeader_1.27mm:PinHeader_1x06_P1.27mm_Vertical -> Connector_PinHeader_1.27mm:PinHeader_1x08_P1.27mm_Horizontal
- renumbered U10 to U4
Connections:
- net +3V3: now also RN1.1 (common)
- net at J3.5 (Pin_5), U4.1 (ROW7): now also RN1.5 (R4)
- net at J3.6 (Pin_6), U4.17 (COL8): now also RN1.6 (R5)
- net at J3.7 (Pin_7), U4.18 (COL9): now also RN1.7 (R6)
- net at J3.4 (Pin_4), U4.2 (ROW6): now also RN1.4 (R3)
- net ~RES: now reaches U4.20 (~Reset)
- net ~RES: now also RN1.8 (R7)
- net at J3.3 (Pin_3), U4.3 (ROW5): now also RN1.3 (R2)
- net at J3.2 (Pin_2), U4.4 (ROW4): now also RN1.2 (R1)
Changed lines of the file:
@@
 EESchema Schematic File Version 4
 LIBS:Raspberry-I2C-LCD-and-Keypad-cache
-EELAYER 29 0
+EELAYER 30 0
 EELAYER END
 $Descr A4 11693 8268
@@
 $EndDescr
 $Comp
-L RasPiInterface:TCA8418 U10
+L RasPiInterface:TCA8418 U4
 U 1 1 5D3B5E8E
 P 4200 2750
-F 0 "U10" H 4150 3531 50  0000 C CNN
+F 0 "U4" H 4150 3531 50  0000 C CNN
 F 1 "TCA8418" H 4150 3440 50  0000 C CNN
 F 2 "Package_DFN_QFN:QFN-24-1EP_4x4mm_P0.5mm_EP2.65x2.65mm" H 4200 2750 50  0001 C CNN
@@
 	3200 2400 3050 2400
 $Comp
-L Connector_Generic:Conn_01x08 J11
+L Connector_Generic:Conn_01x08 J4
 U 1 1 5D3BAFF2
 P 8650 5350
-F 0 "J11" H 8730 5342 50  0000 L CNN
+F 0 "J4" H 8730 5342 50  0000 L CNN
 F 1 "Conn_01x08" H 8730 5251 50  0000 L CNN
-F 2 "Connector_PinHeader_1.27mm:PinHeader_1x06_P1.27mm_Vertical" H 8650 5350 50  0001 C CNN
+F 2 "Connector_PinHeader_1.27mm:PinHeader_1x08_P1.27mm_Horizontal" H 8650 5350 50  0001 C CNN
 F 3 "~" H 8650 5350 50  0001 C CNN
 	1    8650 5350
@@
 Keypad2\n16 Keys
 $Comp
-L Connector_Generic:Conn_01x08 J12
+L Connector_Generic:Conn_01x08 J3
 U 1 1 5D3C4F83
 P 8650 4050
-F 0 "J12" H 8730 4042 50  0000 L CNN
+F 0 "J3" H 8730 4042 50  0000 L CNN
 F 1 "Conn_01x08" H 8730 3951 50  0000 L CNN
-F 2 "Connector_PinHeader_1.27mm:PinHeader_1x06_P1.27mm_Vertical" H 8650 4050 50  0001 C CNN
+F 2 "Connector_PinHeader_1.27mm:PinHeader_1x08_P1.27mm_Horizontal" H 8650 4050 50  0001 C CNN
 F 3 "~" H 8650 4050 50  0001 C CNN
 	1    8650 4050
@@
 GPIO1\n8 IO
 Wire Wire Line
-	4850 2350 6100 2350
-Wire Wire Line
 	4850 2450 6000 2450
 Wire Wire Line
@@
 	4850 3550 7050 3550
 $Comp
-L Connector_Generic:Conn_01x08 J10
+L Connector_Generic:Conn_01x08 J2
 U 1 1 5D3B9F95
 P 8650 2650
-F 0 "J10" H 8730 2642 50  0000 L CNN
+F 0 "J2" H 8730 2642 50  0000 L CNN
 F 1 "Conn_01x08" H 8730 2551 50  0000 L CNN
-F 2 "Connector_PinHeader_1.27mm:PinHeader_1x06_P1.27mm_Vertical" H 8650 2650 50  0001 C CNN
+F 2 "Connector_PinHeader_1.27mm:PinHeader_1x08_P1.27mm_Horizontal" H 8650 2650 50  0001 C CNN
 F 3 "~" H 8650 2650 50  0001 C CNN
 	1    8650 2650
@@
 	5300 3950 5300 5750
 $Comp
-L power:+3.3V #PWR0101
+L power:+3.3V #PWR03
 U 1 1 5D3FD12F
 P 6900 3750
-F 0 "#PWR0101" H 6900 3600 50  0001 C CNN
+F 0 "#PWR03" H 6900 3600 50  0001 C CNN
 F 1 "+3.3V" V 6915 3878 50  0000 L CNN
 F 2 "" H 6900 3750 50  0001 C CNN
@@
 $EndComp
 $Comp
-L power:+3.3V #PWR0102
+L power:+3.3V #PWR02
 U 1 1 5D3FF481
 P 4000 1800
-F 0 "#PWR0102" H 4000 1650 50  0001 C CNN
+F 0 "#PWR02" H 4000 1650 50  0001 C CNN
 F 1 "+3.3V" V 4015 1928 50  0000 L CNN
 F 2 "" H 4000 1800 50  0001 C CNN
@@
 	3850 1800 3850 2050
 Connection ~ 3850 2050
-$Comp
-L Device:R_Network06_US RN1
-U 1 1 5D4089DD
-P 7700 3450
-F 0 "RN1" H 7988 3496 50  0000 L CNN
-F 1 "R_Network06_US" H 7988 3405 50  0000 L CNN
-F 2 "Resistor_THT:R_Array_SIP7" V 8075 3450 50  0001 C CNN
-F 3 "http://www.vishay.com/docs/31509/csc.pdf" H 7700 3450 50  0001 C CNN
-	1    7700 3450
-	1    0    0    -1
-$EndComp
 Wire Wire Line
 	6900 3750 7200 3750
 Wire Wire Line
-	7400 3250 7200 3250
-Wire Wire Line
-	7200 3250 7200 3750
+	7400 3150 7200 3150
 Connection ~ 7200 3750
 Wire Wire Line
@@
 Wire Wire Line
 	4150 4450 8450 4450
-Wire Wire Line
-	7400 3650 7400 3850
 Connection ~ 7400 3850
 Wire Wire Line
 	7400 3850 8450 3850
-Wire Wire Line
-	7500 3650 7500 3950
 Connection ~ 7500 3950
 Wire Wire Line
 	7500 3950 8450 3950
-Wire Wire Line
-	7600 3650 7600 4050
 Connection ~ 7600 4050
 Wire Wire Line
 	7600 4050 8450 4050
-Wire Wire Line
-	7700 3650 7700 4150
 Connection ~ 7700 4150
 Wire Wire Line
 	7700 4150 8450 4150
-Wire Wire Line
-	7800 3650 7800 4250
 Wire Wire Line
 	5000 4250 7800 4250
@@
 Wire Wire Line
 	7800 4250 8450 4250
-Wire Wire Line
-	7900 3650 7900 4350
 Connection ~ 7900 4350
 Wire Wire Line
@@
 	5300 5750 8450 5750
 $Comp
-L Device:C C10
+L Device:C C5
 U 1 1 5D4616B7
 P 3250 4250
-F 0 "C10" H 3365 4296 50  0000 L CNN
+F 0 "C5" H 3365 4296 50  0000 L CNN
 F 1 "100n" H 3365 4205 50  0000 L CNN
-F 2 "Capacitor_THT:C_Disc_D5.0mm_W2.5mm_P2.50mm" H 3288 4100 50  0001 C CNN
+F 2 "Capacitor_THT:C_Disc_D5.0mm_W2.5mm_P5.00mm" H 3288 4100 50  0001 C CNN
 F 3 "~" H 3250 4250 50  0001 C CNN
 	1    3250 4250
@@
 	3250 4450 4150 4450
 $Comp
-L power:+3.3V #PWR0103
+L power:+3.3V #PWR01
 U 1 1 5D465443
 P 3250 4000
-F 0 "#PWR0103" H 3250 3850 50  0001 C CNN
+F 0 "#PWR01" H 3250 3850 50  0001 C CNN
 F 1 "+3.3V" H 3265 4173 50  0000 C CNN
 F 2 "" H 3250 4000 50  0001 C CNN
@@
 Wire Wire Line
 	3250 4100 3250 4000
+$Comp
+L Device:R_Network08_US RN1
+U 1 1 5D3AE6CF
+P 7800 3350
+F 0 "RN1" H 8188 3396 50  0000 L CNN
+F 1 "10k" H 8188 3305 50  0000 L CNN
+F 2 "Resistor_THT:R_Array_SIP9" V 8275 3350 50  0001 C CNN
+F 3 "http://www.vishay.com/docs/31509/csc.pdf" H 7800 3350 50  0001 C CNN
+	1    7800 3350
+	1    0    0    -1
+$EndComp
+Text Label 3050 2950 0    50   ~ 0
+~RES
+Wire Wire Line
+	8000 3650 8400 3650
+Text Label 8250 3650 0    50   ~ 0
+~RES
+Wire Wire Line
+	7200 3150 7200 3750
+Wire Wire Line
+	7400 3550 7400 3850
+Wire Wire Line
+	7500 3550 7500 3950
+Wire Wire Line
+	7600 3550 7600 4050
+Wire Wire Line
+	7700 3550 7700 4150
+Wire Wire Line
+	7800 3550 7800 4250
+Wire Wire Line
+	7900 3550 7900 4350
+Wire Wire Line
+	8000 3550 8000 3650
+Wire Wire Line
+	4850 2350 6100 2350
 $EndSCHEMATC
