File: Raspberry-I2C-LCD-and-Keypad.sch (KiCad schematic (older format))
At the start: 0 parts

Commit message: modified:   DisplayController.sch 	modified:   KeypadController.sch 	new file:   QC2004A.kicad_mod 	modified:   RasPiInterface.lib 	modified:   RasPiInterface.sch 	new file:   Raspberry-I2C-LCD-and-Keypad-B_Cu.gbr 	new file:   Raspberry-I2C-LCD-and-Keypad-B_Mask.gbr 	new file:   Raspberry-I2C-LCD-and-Keypad-B_Paste.gbr 	new file:   Raspberry-I2C-LCD-and-Keypad-Edge_Cuts.gbr 	new file:   Raspberry-I2C-LCD-and-Keypad-F_Cu.gbr 	new file:   Raspberry-I2C-LCD-and-Keypad-F_Mask.gbr 	new file:   Raspberry-I2C-LCD-and-Keypad-F_Paste.gbr 	new file:   Raspberry-I2C-LCD-and-Keypad-F_SilkS.gbr 	new file:   Raspberry-I2C-LCD-and-Keypad-NPTH.drl 	new file:   Raspberry-I2C-LCD-and-Keypad-PTH.drl 	modified:   Raspberry-I2C-LCD-and-Keypad-cache.lib 	modified:   Raspberry-I2C-LCD-and-Keypad.kicad_pcb 	new file:   Raspberry-I2C-LCD-and-Keypad.kicad_pcb-bak 	modified:   Raspberry-I2C-LCD-and-Keypad.pro 	modified:   Raspberry-I2C-LCD-and-Keypad.sch 	modified:   fp-info-cache
Changed lines of the file:
@@
 EESchema Schematic File Version 4
 LIBS:Raspberry-I2C-LCD-and-Keypad-cache
-EELAYER 29 0
+EELAYER 30 0
 EELAYER END
 $Descr A4 11693 8268
@@
 $EndDescr
 $Sheet
-S 4050 1700 2550 2450
+S 4300 2550 2550 2450
 U 5D399320
 F0 "DisplayController" 50
 F1 "DisplayController.sch" 50
+F2 "5V" I L 4300 2700 50
+F3 "3.3V" I L 4300 2850 50
+F4 "GND" I L 4300 3850 50
+F5 "SDA" I L 4300 3050 50
+F6 "SCL" I L 4300 3250 50
+F7 "SDG" I L 4300 3150 50
 $EndSheet
 $Sheet
-S 1850 1650 1400 2450
+S 2100 2500 1400 2450
 U 5D399389
 F0 "RasPiInterface" 50
 F1 "RasPiInterface.sch" 50
-F2 "5V" I R 3250 1850 50
-F3 "3.3V" I R 3250 2000 50
-F4 "SDA" I R 3250 2200 50
-F5 "SCL" I R 3250 2400 50
-F6 "~iNT" I R 3250 2600 50
-F7 "GND" I R 3250 3000 50
-F8 "SDG" I R 3250 2300 50
+F2 "5V" I R 3500 2700 50
+F3 "3.3V" I R 3500 2850 50
+F4 "SDA" I R 3500 3050 50
+F5 "SCL" I R 3500 3250 50
+F6 "~iNT" I R 3500 3450 50
+F7 "GND" I R 3500 3850 50
+F8 "SDG" I R 3500 3150 50
 $EndSheet
 Wire Wire Line
-	7600 2000 7400 2000
+	7850 2850 7650 2850
 Wire Wire Line
-	3400 2000 3250 2000
+	3650 2850 3500 2850
 Wire Wire Line
-	3400 1100 7400 1100
+	3650 1950 7650 1950
 Wire Wire Line
-	7600 2200 7300 2200
+	7850 3050 7550 3050
 Wire Wire Line
-	7300 1200 3500 1200
+	7550 2050 3750 2050
 Wire Wire Line
-	3500 2200 3250 2200
+	3750 3050 3500 3050
 Wire Wire Line
-	7100 2400 7600 2400
+	7350 3250 7850 3250
 $Sheet
-S 7600 1750 2400 2400
+S 7850 2600 2400 2400
 U 5D399061
 F0 "KeypadController" 50
 F1 "KeypadController.sch" 50
-F2 "SDA" I L 7600 2200 50
-F3 "SCL" I L 7600 2400 50
-F4 "~INT" I L 7600 2500 50
-F5 "3.3V" I L 7600 2000 50
-F6 "GND" I L 7600 2800 50
-F7 "SDG" I L 7600 2300 50
+F2 "SDA" I L 7850 3050 50
+F3 "SCL" I L 7850 3250 50
+F4 "~INT" I L 7850 3350 50
+F5 "3.3V" I L 7850 2850 50
+F6 "GND" I L 7850 3650 50
+F7 "SDG" I L 7850 3150 50
 $EndSheet
 Wire Wire Line
-	7000 2500 7600 2500
+	7250 3350 7850 3350
 Wire Wire Line
-	7600 2300 7200 2300
+	7850 3150 7450 3150
 Wire Wire Line
-	7300 1200 7300 2200
+	7550 2050 7550 3050
 Wire Wire Line
-	7400 1100 7400 2000
+	7650 1950 7650 2850
 Wire Wire Line
-	3500 1200 3500 2200
+	3750 2050 3750 3050
 Wire Wire Line
-	3400 1100 3400 2000
+	3650 1950 3650 2850
 Wire Wire Line
-	3250 2600 3800 2600
+	3500 3450 4050 3450
 Wire Wire Line
-	3250 2400 3700 2400
+	3500 3250 3950 3250
 Wire Wire Line
-	3250 2300 3600 2300
+	3500 3150 3850 3150
 Wire Wire Line
-	3800 1500 3800 2600
+	4050 2350 4050 3450
 Wire Wire Line
-	3700 1400 3700 2400
+	3950 2250 3950 3250
 Wire Wire Line
-	3600 1300 3600 2300
+	3850 2150 3850 3150
 Wire Wire Line
-	7200 1300 7200 2300
+	7450 2150 7450 3150
 Wire Wire Line
-	7100 1400 7100 2400
+	7350 2250 7350 3250
 Wire Wire Line
-	7000 1500 7000 2500
+	7250 2350 7250 3350
 Wire Wire Line
-	3800 1500 7000 1500
+	4050 2350 7250 2350
 Wire Wire Line
-	3700 1400 7100 1400
+	3950 2250 7350 2250
 Wire Wire Line
-	3600 1300 7200 1300
+	3850 2150 7450 2150
 Wire Wire Line
-	3250 3000 3800 3000
+	3500 3850 4050 3850
 Wire Wire Line
-	3800 3000 3800 4650
+	4050 3850 4050 5500
 Wire Wire Line
-	3800 4650 7000 4650
+	4050 5500 7250 5500
 Wire Wire Line
-	7000 4650 7000 2800
+	7250 5500 7250 3650
 Wire Wire Line
-	7000 2800 7600 2800
+	7250 3650 7850 3650
+Wire Wire Line
+	3500 2700 4300 2700
+Wire Wire Line
+	4300 2850 3650 2850
+Connection ~ 3650 2850
+Wire Wire Line
+	4300 3850 4050 3850
+Connection ~ 4050 3850
+Wire Wire Line
+	4300 3050 3750 3050
+Connection ~ 3750 3050
+Wire Wire Line
+	4300 3250 3950 3250
+Connection ~ 3950 3250
+Wire Wire Line
+	4300 3150 3850 3150
+Connection ~ 3850 3150
 $EndSCHEMATC
